File: SX1262_LoRa_Module/SX1262_LoRa_Module.kicad_sch (KiCad schematic)
At the start: 33 parts, among them J1 Conn_01x10_Pin, Q1 32.0Mhz, U1 SX1262IMLTRT, U2 PE4259

Commit message: -added side castellation
-added side castellation
Parts:
- added J2, J3: Conn_01x10_Pin, Connector_PinHeader_2.54mm:PinHeader_1x10_P2.54mm_Vertical, symbol Connector:Conn_01x10_Pin
Connections:
- net GND: now also J2.1 (Pin_1), J2.10 (Pin_10), J2.2 (Pin_2), J2.3 (Pin_3), J2.4 (Pin_4), J2.5 (Pin_5), J2.6 (Pin_6), J2.7 (Pin_7), J2.8 (Pin_8), J2.9 (Pin_9), J3.1 (Pin_1), J3.10 (Pin_10), J3.2 (Pin_2), J3.3 (Pin_3), J3.4 (Pin_4), J3.5 (Pin_5), J3.6 (Pin_6), J3.7 (Pin_7), J3.8 (Pin_8), J3.9 (Pin_9)

Commit message: -update bom
-updated bom based on the evm
-put booklet list for the inductor
Parts:
- C1: LCSC (none) -> C307434
- C10, C9: LCSC (none) -> C76906
- C11: LCSC (none) -> C48346
- C12, C7: LCSC (none) -> C1553
- C14, C15: LCSC (none) -> C189467
- C16: LCSC (none) -> C14445
- C17: LCSC (none) -> C92361
- C18: LCSC (none) -> C1525
- C19: LCSC (none) -> C53282223
- C2: LCSC (none) -> C76970
- C4: LCSC (none) -> C88891
- C5: LCSC (none) -> C161329
- C6, C8: LCSC (none) -> C1563
- L2: LCSC (none) -> C106231
- R3, R4: LCSC (none) -> C106232
Changed lines of the file:
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@@
 			)
 		)
+		(property "LCSC" "C1525"
+			(at 124.243 118.3821 0)
+			(effects
+				(font
+					(size 1.27 1.27)
+				)
+				(hide yes)
+			)
+		)
 		(pin "2"
 		)
@@
 			)
 		)
+		(property "LCSC" "C1553"
+			(at 215.6505 121.8641 0)
+			(effects
+				(font
+					(size 1.27 1.27)
+				)
+				(hide yes)
+			)
+		)
 		(pin "2"
 		)
@@
 			)
 		)
+		(property "LCSC" "C76906"
+			(at 314.9367 95.8427 0)
+			(effects
+				(font
+					(size 1.27 1.27)
+				)
+				(hide yes)
+			)
+		)
 		(pin "2"
 		)
@@
 			)
 		)
+		(property "LCSC" "C14445"
+			(at 137.9265 78.5803 0)
+			(effects
+				(font
+					(size 1.27 1.27)
+				)
+				(hide yes)
+			)
+		)
 		(pin "2"
 		)
@@
 			)
 		)
+		(property "LCSC" "C1563"
+			(at 305.7108 92.0327 90)
+			(effects
+				(font
+					(size 1.27 1.27)
+				)
+				(hide yes)
+			)
+		)
 		(pin "2"
 		)
@@
 			)
 		)
+		(property "LCSC" "C53282223"
+			(at 165.698 169.7263 0)
+			(effects
+				(font
+					(size 1.27 1.27)
+				)
+				(hide yes)
+			)
+		)
 		(pin "2"
 		)
@@
 			)
 		)
+		(property "LCSC" "C1563"
+			(at 235.8552 80.459 90)
+			(effects
+				(font
+					(size 1.27 1.27)
+				)
+				(hide yes)
+			)
+		)
 		(pin "2"
 		)
@@
 			)
 		)
+		(property "LCSC" "C48346"
+			(at 224.7945 102.8141 90)
+			(effects
+				(font
+					(size 1.27 1.27)
+				)
+				(hide yes)
+			)
+		)
 		(pin "2"
 		)
@@
 			)
 		)
+		(property "LCSC" "C92361"
+			(at 112.0945 118.4621 0)
+			(effects
+				(font
+					(size 1.27 1.27)
+				)
+				(hide yes)
+			)
+		)
 		(pin "2"
 		)
@@
 			)
 		)
+		(property "LCSC" "C76906"
+			(at 334.6757 95.8427 0)
+			(effects
+				(font
+					(size 1.27 1.27)
+				)
+				(hide yes)
+			)
+		)
 		(pin "2"
 		)
@@
 			)
 		)
+		(property "LCSC" "C307434"
+			(at 194.8225 66.3461 0)
+			(effects
+				(font
+					(size 1.27 1.27)
+				)
+				(hide yes)
+			)
+		)
 		(pin "2"
 		)
@@
 			)
 		)
+		(property "LCSC" "C88891"
+			(at 225.3411 74.8905 90)
+			(effects
+				(font
+					(size 1.27 1.27)
+				)
+				(hide yes)
+			)
+		)
 		(pin "2"
 		)
@@
 			)
 		)
+		(property "LCSC" "C161329"
+			(at 232.0452 84.269 0)
+			(effects
+				(font
+					(size 1.27 1.27)
+				)
+				(hide yes)
+			)
+		)
 		(pin "2"
 		)
@@
 			)
 		)
+		(property "LCSC" "C106231"
+			(at 201.8245 80.459 90)
+			(effects
+				(font
+					(size 1.27 1.27)
+				)
+				(hide yes)
+			)
+		)
 		(pin "2"
 		)
@@
 			)
 		)
+		(property "LCSC" "C106232"
+			(at 284.0346 120.8481 90)
+			(effects
+				(font
+					(size 1.27 1.27)
+				)
+				(hide yes)
+			)
+		)
 		(pin "1"
 		)
@@
 			)
 		)
+		(property "LCSC" "C76970"
+			(at 203.0265 66.2381 0)
+			(effects
+				(font
+					(size 1.27 1.27)
+				)
+				(hide yes)
+			)
+		)
 		(pin "2"
 		)
@@
 			)
 		)
-		(property "LCSC" ""
+		(property "LCSC" "C1553"
 			(at 258.3985 84.5261 0)
 			(effects
@@
 			)
 		)
+		(property "LCSC" "C106232"
+			(at 286.0085 59.1261 90)
+			(effects
+				(font
+					(size 1.27 1.27)
+				)
+				(hide yes)
+			)
+		)
 		(pin "1"
 		)
@@
 			)
 		)
+		(property "LCSC" "C189467"
+			(at 293.6384 127.4319 0)
+			(effects
+				(font
+					(size 1.27 1.27)
+				)
+				(hide yes)
+			)
+		)
 		(pin "2"
 		)
@@
 			)
 		)
-		(property "Field5" ""
+		(property "LCSC" "C189467"
 			(at 294.4691 62.9361 0)
 			(effects
